Commit message: Initial upload from VM

File: fr5_description/urdf/fr5v6.urdf (robot description, URDF)
Before this commit: robot fr5v6, 11 links, 10 joints
Links:
- added link camera_link, mass 0.01; collision box size=0.04 0.04 0.02; visual box size=0.04 0.04 0.02
Joints:
- added joint camera_joint: type fixed, parent hand_base_link, child camera_link, origin xyz=-0.05 0.03 0.1 rpy=0 -1.5708 0
